Commit message: added optimazatation

File: m2wr_description/urdf/m2wr.xacro (robot description, xacro)
@@ -58,5 +58,5 @@
       <origin xyz="0 0 0" rpy="0 0 0" />
       <geometry>
-        <cylinder radius="0.05" length="0.1"/>
+        <cylinder radius="0.05" length="0.2"/>
       </geometry>
       <material name="white" />
@@ -65,12 +65,37 @@
       <origin xyz="0 0 0" rpy="0 0 0"/>
       <geometry>
-        <cylinder radius="0.05" length="0.1"/>
+        <cylinder radius="0.05" length="0.2"/>
       </geometry>
     </collision>
   </link>
   <joint name="joint_sensor_laser" type="fixed">
-    <origin xyz="0.15 0 0.05" rpy="0 0 0"/>
+    <origin xyz="0.15 0 0.1" rpy="0 0 0"/>
     <parent link="link_chassis"/>
     <child link="sensor_laser"/>
+  </joint>
+  <link name="camera_box">
+    <inertial>
+      <mass value="0.5"/>
+      <origin rpy="0 0 0" xyz="0 0 0"/>
+      <inertia ixx="0.000002083" ixy="0" ixz="0" iyy="0.000002083" iyz="0" izz="0.000002083"/>
+    </inertial>
+    <!-- body -->
+    <collision name="camera_box_collision">
+      <geometry>
+        <box size="0.005 0.05 0.05"/>
+      </geometry>
+    </collision>
+    <visual>
+      <origin rpy="0 0 0" xyz="0 0 0"/>
+      <geometry>
+        <box size="0.005 0.05 0.05"/>
+      </geometry>
+      <material name="blue"/>
+    </visual>
+  </link>
+  <joint name="joint_camera_box" type="fixed">
+    <origin xyz="0.25 0 0" rpy="0 0 0" />
+    <parent link="link_chassis" />
+    <child link="camera_box"/>
   </joint>
   <xacro:link_wheel name="link_right_wheel" />
